File: designs/hardware/bGeigieCast V1.6.0(StampS3)/bGeigieCast V1.6.0(StampS3)/bGeigieCast V1.6.0(StampS3).kicad_pcb (KiCad board)
At the start: 2 copper layers, 25.2 x 28.4 mm, 3 parts, among them J1 Left, J2 Right, U2 XBEE-socket

Commit message: Updated and cleaned out the board
Routing:
- added copper zone on B.Cu, net GND
- added copper zone on F.Cu, net GND
Other:
- board size 25.2 x 28.4 mm -> 25.2 x 28.5 mm
- board text added: "bGeigieCast V1.6.2 safecast 2024"
- board text removed: "bGeigieCast V1.6.2 safecast 2023"
