File: designs/hardware/bGeigieCast V1.6.0(StampS3)/bGeigieCast V1.6.0(StampS3)/bGeigieCast V1.6.0(StampS3).kicad_sch (KiCad schematic)
At the start: 3 parts, among them J1 Left, J2 Right, U2 XBEE-socket

Commit message: Updated and cleaned out the board
Other:
- note added: "bGeigieCast M5stack Stamp V1.6.2"
- note removed: "V1.1"
- note removed: "bGeigieCast M5stack Stamp V1.6.1"
